Commit message: made arm telescoping

File: models/morpheus_description/morpheus.urdf (robot description, URDF)
Before this commit: robot morpheus, 7 links, 6 joints
Links:
- link arm1: geometry collision box size=0.05 0.05 0.3; visual box size=0.075 0.075 0.3
- link arm2: geometry collision box size=0.07 0.07 0.3; visual box size=0.07 0.07 0.3
- link arm3: geometry collision box size=0.06 0.06 0.3; visual box size=0.06 0.06 0.3
- link arm5: geometry collision box size=0.04 0.04 0.3; visual box size=0.04 0.04 0.3

Commit message: created morpheus urdf

File: models/morpheus_description/morpheus.urdf (robot description, URDF)
Before this commit: robot morpheus, 7 links, 6 joints
Links:
- added link gripper_base, mass .01; collision box size=0.01 0.2 0.03; visual box size=0.01 0.2 0.03
- added link left_gripper, mass .01; collision mesh filename=left_gripper.stl scale=1 1 1; visual mesh filename=left_gripper.stl scale=1 1 1
- added link right_gripper, mass .01; collision mesh filename=right_gripper.stl scale=1 1 1; visual mesh filename=right_gripper.stl scale=1 1 1
- added link wrist, mass .01; collision box size=0.07 0.07 0.07; visual box size=0.04 0.04 0.04
Joints:
- added joint arm5_to_wrist: type continuous, parent arm5, child wrist, axis 0 0 1, limit lower=-0.25 upper=0.25 effort=300 velocity=10
- added joint gripper_base_to_left_gripper: type fixed, parent gripper_base, child left_gripper
- added joint gripper_base_to_right_gripper: type fixed, parent gripper_base, child right_gripper
- added joint wrist_to_gripper_base: type fixed, parent wrist, child gripper_base
