Commit message: arm fully works

File: models/morpheus_description/morpheus_rigid.urdf (robot description, URDF)
Before this commit: robot morpheus, 11 links, 10 joints
Joints:
- joint arm5_to_wrist: limit lower=-3.14 upper=3.14 effort=300 velocity=10 -> lower=-0.25 upper=0.25 effort=1 velocity=10; origin xyz=0.28 0 -0.54 rpy=0 0 0 -> (none)
- joint gripper_base_to_left_gripper: axis 1 0 0 -> (none); limit lower=0.0 upper=0.06 effort=300 velocity=10 -> (none); origin xyz=0.062 0.06 -0.011 rpy=0. 0 -1.57 -> (none); type prismatic -> fixed
- joint gripper_base_to_right_gripper: axis 1 0 0 -> (none); limit lower=-0.06 upper=0.0 effort=300 velocity=10 -> (none); origin xyz=0.062 -0.06 -0.011 rpy=0. 0 -1.57 -> (none); type prismatic -> fixed
- joint wrist_to_gripper_base: origin xyz=0.02 0 -0.01 rpy=0 0.86 0 -> (none)
