Commit message: stretch on husky (morph) fully implemented

File: models/morpheus_description/husky_with_morph.urdf (robot description, URDF)
Before this commit: robot husky_robot, 12 links, 11 joints
Links:
- added link arm1, mass .01; collision box size=0.05 0.05 0.3; visual box size=0.075 0.075 0.3
- added link arm2, mass .01; collision box size=0.07 0.07 0.3; visual box size=0.07 0.07 0.3
- added link arm3, mass .01; collision box size=0.06 0.06 0.3; visual box size=0.06 0.06 0.3
- added link arm4, mass .01; collision box size=0.05 0.05 0.3; visual box size=0.05 0.05 0.3
- added link arm5, mass .01; collision box size=0.04 0.04 0.3; visual box size=0.04 0.04 0.3
- added link gripper_base, mass .01; collision box size=0.01 0.2 0.03; visual box size=0.01 0.2 0.03
- added link head, mass .01; collision box size=0.05 0.05 0.15; visual box size=0.05 0.05 0.15
- added link left_gripper, mass .01; collision mesh filename=left_gripper.stl scale=1 1 1; visual mesh filename=left_gripper.stl scale=1 1 1
- added link right_gripper, mass .01; collision mesh filename=right_gripper.stl scale=1 1 1; visual mesh filename=right_gripper.stl scale=1 1 1
- added link spine, mass .01; collision box size=0.05 0.05 1.8; visual box size=0.05 0.05 1.8
- added link wrist, mass .01; collision box size=0.07 0.07 0.07; visual box size=0.04 0.04 0.04
- link platform_link: geometry collision box size=0.3 0.3 0.1; visual box size=0.3 0.3 0.1
Joints:
- added joint arm1_to_arm2: type prismatic, parent arm1, child arm2, origin xyz=0 0 0 rpy=0 0 0, axis 1 0 0, limit lower=0.0 upper=0.25 effort=10 velocity=0.25
- added joint arm2_to_arm3: type prismatic, parent arm2, child arm3, origin xyz=0 0 0 rpy=0 0 0, axis 1 0 0, limit lower=0.0 upper=0.25 effort=10 velocity=0.25
- added joint arm3_to_arm4: type prismatic, parent arm3, child arm4, origin xyz=0 0 0 rpy=0 0 0, axis 1 0 0, limit lower=0.0 upper=0.25 effort=10 velocity=0.25
- added joint arm4_to_arm5: type prismatic, parent arm4, child arm5, origin xyz=0 0 0 rpy=0 0 0, axis 1 0 0, limit lower=0.0 upper=0.25 effort=10 velocity=0.25
- added joint arm5_to_wrist: type revolute, parent arm5, child wrist, origin xyz=0.28 0 -0.54 rpy=0 0 0, axis 0 0 1, limit lower=-3.14 upper=3.14 effort=300 velocity=10
- added joint gripper_base_to_left_gripper: type prismatic, parent gripper_base, child left_gripper, origin xyz=0.062 0.06 -0.011 rpy=0. 0 -1.57, axis 1 0 0, limit lower=0.0 upper=0.06 effort=300 velocity=10
- added joint gripper_base_to_right_gripper: type prismatic, parent gripper_base, child right_gripper, origin xyz=0.062 -0.06 -0.011 rpy=0. 0 -1.57, axis 1 0 0, limit lower=-0.06 upper=0.0 effort=300 velocity=10
- added joint morph_to_husky: type fixed, parent platform_link, child spine, origin xyz=0 0 1. rpy=0 0 -1.57
- added joint spine_to_arm1: type prismatic, parent spine, child arm1, origin xyz=0 0 0 rpy=0 0 0, axis 0 0 1, limit lower=0.0 upper=1.3 effort=10 velocity=0.25
- added joint spine_to_head: type fixed, parent spine, child head
- added joint wrist_to_gripper_base: type fixed, parent wrist, child gripper_base, origin xyz=0.02 0 -0.01 rpy=0 0.86 0
