Commit message: autonomous open top right drawer working

File: models/morpheus_description/morph_with_horizontal_gripper.urdf (robot description, URDF)
Before this commit: robot husky_robot, 23 links, 22 joints
Links:
- added link hook, mass .01; collision mesh filename=hook.stl scale=1 1 1; visual mesh filename=hook.stl scale=1 1 1
Joints:
- added joint hook_to_wrist: type fixed, parent wrist, child hook, origin xyz=-0.06 0 -0.01 rpy=1.57 -0 3.14

Commit message: about to start food preparation

File: models/morpheus_description/morph_with_horizontal_gripper.urdf (robot description, URDF)
Before this commit: robot husky_robot, 24 links, 23 joints
Joints:
- joint arm5_to_wrist: limit lower=-3.14 upper=3.14 effort=300 velocity=10 -> (none); type revolute -> fixed
- joint wrist_to_gripper_base: type revolute -> fixed

Commit message: cooking task preparation

File: models/morpheus_description/morph_with_horizontal_gripper.urdf (robot description, URDF)
Before this commit: robot husky_robot, 24 links, 23 joints
Joints:
- joint arm5_to_wrist: limit (none) -> lower=-3.14 upper=3.14 effort=12000 velocity=2.61

Commit message: repaired vertical twist joint parameters

File: models/morpheus_description/morph_with_horizontal_gripper.urdf (robot description, URDF)
Before this commit: robot husky_robot, 24 links, 23 joints
Links:
- link gripper_base: mass .01 -> .2
- link wrist: mass .01 -> .2
Joints:
- joint arm5_to_wrist: limit lower=-3.14 upper=3.14 effort=12000 velocity=2.61 -> lower=-3.14 upper=3.14 effort=12 velocity=2.61
- joint wrist_to_gripper_base: limit lower=-3.14 upper=3.14 effort=300 velocity=10 -> lower=-3.14 upper=3.14 effort=12 velocity=2.61; type fixed -> revolute
